File: bt_bio.brd (EAGLE design)
At the start: 57.8 x 57.9 mm, 74 parts, among them U1 ADP121-AUJZ33R7, U2 MCP73837-FCI/UN, U4 ADP121-AUJZ18R7, U5 LSM9DS1, X1 53047-03, X2 MINI-USB-SHIELD-UX60-MB-5ST, X3 53047-03

Commit message: Version European Circiuts
Parts:
- C29: device rcl:C1206 -> rcl:C0603
- R2: value 2K2 -> 2.2K
- moved VBAT 1.73 mm to (41.7, 35.7)
- moved R2 1.15 mm to (46.4, 37.3)
Routing:
- net N$31: track 112.4 -> 110.6 mm
- net V+: track 200.3 -> 201.7 mm
- net N$17: track 1.82 -> 2.97 mm
- net N$6: track 5.95 -> 4.80 mm
- net GND: vias 40 -> 39
Changed lines of the file:
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@@
 </element>
 <element name="LED1" library="led" package="CHIPLED_0805" value="BLUE" x="46.357" y="34.344" rot="R270"/>
-<element name="R2" library="rcl" package="R0603" value="2K2" x="46.448" y="36.156"/>
+<element name="R2" library="rcl" package="R0603" value="2.2K" x="46.373" y="37.306"/>
 <element name="C10" library="rcl" package="C0603" value="100nF" x="32.739" y="32.163" smashed="yes" rot="R180">
 <attribute name="NAME" x="30.459" y="32.843" size="1.27" layer="25" rot="R180"/>
@@
 <element name="R19" library="rcl" package="R0603" value="2.2K" x="40.85" y="22" rot="R180"/>
 <element name="R20" library="resistor" package="R0603" value="33K" x="42.1" y="19.95" rot="R180"/>
-<element name="VBAT" library="jumper" package="JP1" value="Vbat" x="41.775" y="37.4" smashed="yes">
-<attribute name="NAME" x="44.674" y="35.31" size="1.27" layer="25" ratio="10" rot="R90"/>
-<attribute name="VALUE" x="44.696" y="34.86" size="1.27" layer="27" ratio="10" rot="R90"/>
+<element name="VBAT" library="jumper" package="JP1" value="Vbat" x="41.725" y="35.675" smashed="yes">
+<attribute name="NAME" x="44.624" y="33.585" size="1.27" layer="25" ratio="10" rot="R90"/>
+<attribute name="VALUE" x="44.646" y="33.135" size="1.27" layer="27" ratio="10" rot="R90"/>
 </element>
 <element name="R21" library="rcl" package="R0603" value="2.2K" x="43.775" y="28.4" rot="R270"/>
@@
 <element name="C24" library="rcl" package="C1206" value="10uF" x="38" y="22.225" rot="R270"/>
 <element name="U$1" library="rn4678" package="RN4678" value="RN4678" x="34.875" y="53.4" rot="R270"/>
-<element name="C29" library="rcl" package="C1206" value="1uF" x="42.975" y="55.4" smashed="yes" rot="R180">
-<attribute name="NAME" x="39.295" y="56.082" size="1.27" layer="25" rot="R180"/>
+<element name="C29" library="rcl" package="C0603" value="1uF" x="42.975" y="55.4" smashed="yes" rot="R180">
+<attribute name="NAME" x="39.895" y="56.157" size="1.27" layer="25" rot="R180"/>
 <attribute name="VALUE" x="44.245" y="57.813" size="1.27" layer="27" rot="R180"/>
 </element>
@@
 <contactref element="X2" pad="M3"/>
 <contactref element="X2" pad="M4"/>
-<via x="39.628" y="33.976" extent="1-16" drill="0.6" shape="octagon"/>
 <via x="29.528" y="45.876" extent="1-16" drill="0.6" shape="octagon"/>
 <via x="29.378" y="52.026" extent="1-16" drill="0.6" shape="octagon"/>
@@
 <contactref element="C29" pad="2"/>
 <via x="33.678" y="45.201" extent="1-16" drill="0.6" shape="octagon"/>
-<via x="39.828" y="55.451" extent="1-16" drill="0.6" shape="octagon"/>
+<via x="40.528" y="55.476" extent="1-16" drill="0.6" shape="octagon"/>
 <via x="46.553" y="40.051" extent="1-16" drill="0.6" shape="octagon"/>
 <via x="51.053" y="54.201" extent="1-16" drill="0.6" shape="octagon"/>
@@
 <wire x1="33.201" y1="33.876" x2="33.251" y2="33.907" width="0.254" layer="1"/>
 <via x="36.85" y="31.35" extent="1-16" drill="0.6" shape="octagon"/>
-<via x="47.6" y="56.925" extent="1-16" drill="0.6" shape="octagon"/>
-<wire x1="47.6" y1="56.925" x2="48.2" y2="57.175" width="0.254" layer="16"/>
+<via x="47.6" y="55.175" extent="1-16" drill="0.6" shape="octagon"/>
+<wire x1="47.6" y1="55.175" x2="48.2" y2="57.175" width="0.254" layer="16"/>
 <wire x1="48.75" y1="33" x2="46.5000375" y2="33.009621875" width="0.254" layer="16"/>
 <wire x1="46.5000375" y1="33.009621875" x2="36.85" y2="32.95" width="0.254" layer="16"/>
@@
 <contactref element="U1" pad="5"/>
 <wire x1="27.6" y1="57.15" x2="47.6" y2="57.175" width="0.254" layer="1"/>
-<wire x1="47.6" y1="57.175" x2="47.6" y2="56.925" width="0.254" layer="1"/>
+<wire x1="47.6" y1="57.175" x2="47.6" y2="55.175" width="0.254" layer="1"/>
 <wire x1="20.688" y1="44.286" x2="20.7" y2="48.211" width="0.254" layer="1"/>
 <wire x1="20.7" y1="48.211" x2="25.25" y2="50.15" width="0.254" layer="1"/>
@@
 <wire x1="31.79" y1="28.535" x2="33" y2="27.325" width="0.254" layer="1"/>
 <contactref element="U$1" pad="4"/>
-<wire x1="47.6" y1="56.925" x2="47.65" y2="55" width="0.254" layer="1"/>
+<wire x1="47.6" y1="55.175" x2="47.65" y2="55" width="0.254" layer="1"/>
 <wire x1="47.65" y1="55" x2="47.65" y2="54.575" width="0.254" layer="1"/>
 <wire x1="47.65" y1="54.575" x2="47.675" y2="52.9" width="0.254" layer="1"/>
@@
 <contactref element="LED1" pad="C"/>
 <contactref element="R2" pad="2"/>
-<wire x1="47.298" y1="36.156" x2="47.407" y2="34.344" width="0.254" layer="1"/>
+<wire x1="47.223" y1="37.306" x2="47.407" y2="34.344" width="0.254" layer="1"/>
 </signal>
 <signal name="SPI_MISO">
@@
 <wire x1="38" y1="24.225" x2="38" y2="23.625" width="0.4064" layer="1"/>
 <wire x1="40.35" y1="31" x2="41.75" y2="31.95" width="0.254" layer="1"/>
-<wire x1="41.75" y1="31.95" x2="41.775" y2="36.13" width="0.254" layer="1"/>
+<wire x1="41.75" y1="31.95" x2="41.725" y2="34.405" width="0.254" layer="1"/>
 </signal>
 <signal name="N$25">
@@
 <wire x1="45.475" y1="52.9" x2="44.375" y2="52.9" width="0.254" layer="1"/>
 <contactref element="C29" pad="1"/>
-<wire x1="44.375" y1="55.4" x2="44.375" y2="52.9" width="0.254" layer="1"/>
+<wire x1="43.825" y1="55.4" x2="44.375" y2="52.9" width="0.254" layer="1"/>
 </signal>
 <signal name="N$6">
 <contactref element="R2" pad="1"/>
 <contactref element="U$1" pad="30"/>
-<wire x1="45.598" y1="36.156" x2="45.523" y2="40.977" width="0.254" layer="1"/>
+<wire x1="45.523" y1="37.306" x2="45.523" y2="40.977" width="0.254" layer="1"/>
 <wire x1="45.523" y1="40.977" x2="45.5" y2="41.625" width="0.254" layer="1"/>
 <wire x1="45.5" y1="41.625" x2="45.5" y2="41.525" width="0.254" layer="1"/>
